File: pcb/digital_compass/digital_compass.kicad_sch (KiCad schematic)
At the start: 10 parts, among them SW1 SW_SPDT, U1 L7805, U2 Seeed Studio XIAO SAMD21, U3 Level_Shifter, U4 QMC5883L, U5 Adafruit_Neopixel_Ring_24

Commit message: Fix power switch and update schematic/pcb/gerbers.
Turns out the L7805 consumes power when connected to an input power
source even if the output is disconnected. We therefore move the power
switch to the input side of the regulator to prevent power consumption
when the compass is turned off.
Connections:
- net +9V: now also SW1.2 (B); no longer C1.1, U1.1 (IN)
- net at C2.1, U1.3 (OUT): now also U2.14 (5V), U3.10 (HV), U4.1 (VCC), U5.1 (PWR1), U5.2 (PWR2); no longer SW1.2 (B)
- new net: C1.1, SW1.1 (A), U1.1 (IN)
Other:
- moved on the sheet: BT1, SW1
